Commit message: Fix pusher0 rotation

File: ur5_push_setup/urdf/arm.urdf.xacro (robot description, xacro)
@@ -67,5 +67,5 @@
 	  <parent link="pusher"/>
 	  <child link="pusher0"/>
-	  <origin xyz="0.0 0.17 0.0" rpy="0.0 0.0 0.0" />
+	  <origin xyz="0.0 0.17 0.0" rpy="0.0 0.0 ${pi/2}" />
   </joint>
 </robot>

Commit message: Use version 2 of applicable pusher

File: ur5_push_setup/urdf/arm.urdf.xacro (robot description, xacro)
@@ -48,5 +48,5 @@
 	  <visual>
 		  <geometry>
-			  <mesh filename="package://ur5_push_setup/meshes/visual/pusher_1_binary.stl" scale="0.001 0.001 0.001"/>
+			  <mesh filename="package://ur5_push_setup/meshes/visual/pusher_2_binary.stl" scale="0.001 0.001 0.001"/>
 		  </geometry>
 		  <material name="gray"/>
@@ -54,5 +54,5 @@
 	  <collision>
 		  <geometry>
-			  <mesh filename="package://ur5_push_setup/meshes/collision/pusher_1_binary.stl" scale="0.001 0.001 0.001"/>
+			  <mesh filename="package://ur5_push_setup/meshes/collision/pusher_2_binary.stl" scale="0.001 0.001 0.001"/>
 		  </geometry>
 	  </collision>
@@ -61,5 +61,5 @@
 	  <parent link="s_model_palm"/>
 	  <child link="pusher"/>
-	  <origin xyz="0.0 0.0305 0.0" rpy="0.0 0.0 0.0" />
+	  <origin xyz="0.0 0.05625 0.0" rpy="0.0 0.0 0.0" />
   </joint>
   <link name="pusher0"/>
@@ -67,5 +67,5 @@
 	  <parent link="pusher"/>
 	  <child link="pusher0"/>
-	  <origin xyz="0.0 0.17 0.0" rpy="0.0 0.0 ${pi/2}" />
+	  <origin xyz="0.0 0.2 0.0" rpy="0.0 0.0 ${pi/2}" />
   </joint>
 </robot>
