Commit message: Use original arm description
Since the hardware is used with multiple modifications there exist many
attached devices that are represented in the description.
It is easier to just append the pusher to the original arm description
than copying it each time there is a change.
The tams_ur5_setup.urdf.xacro now attaches the pusher link.

File: ur5_push_setup/urdf/tams_ur5_setup.urdf.xacro (robot description, xacro)
@@ -6,5 +6,6 @@
   <xacro:include filename="$(find tams_ur5_setup_description)/urdf/tams_corner.urdf.xacro" />
   <!-- arm -->
-  <xacro:include filename="$(find ur5_push_setup)/urdf/arm.urdf.xacro" />
+  <xacro:include filename="$(find tams_ur5_description)/urdf/arm.urdf.xacro" />
+  <xacro:include filename="$(find ur5_push_setup)/urdf/pusher.urdf.xacro" />
   <link name="world" />
   <joint name="world_floor_joint" type="fixed">
@@ -24,3 +25,7 @@
     <origin xyz="0 0 0.003" rpy="0.0 0.0 ${pi/2}" />
   </joint>
+  <!-- pusher attachemenet -->
+  <xacro:pusher name="pusher" parent="s_model_palm" >
+    <origin xyz="0.0 0.05625 0.0" rpy="0.0 0.0 0.0" />
+  </xacro:pusher>
 </robot>
