Commit message: Use short package names

File: bringup/urdf/pusher.urdf.xacro (robot description, xacro)
@@ -8,5 +8,5 @@
 	  <visual>
 		  <geometry>
-			  <mesh filename="package://ur5_push_setup/meshes/visual/pusher_2_binary.stl" scale="0.001 0.001 0.001"/>
+			  <mesh filename="package://tams_ur5_push_bringup/meshes/visual/pusher_2_binary.stl" scale="0.001 0.001 0.001"/>
 		  </geometry>
 		  <material name="gray"/>
@@ -14,5 +14,5 @@
 	  <collision>
 		  <geometry>
-			  <mesh filename="package://ur5_push_setup/meshes/collision/pusher_2_binary.stl" scale="0.001 0.001 0.001"/>
+			  <mesh filename="package://tams_ur5_push_bringup/meshes/collision/pusher_2_binary.stl" scale="0.001 0.001 0.001"/>
 		  </geometry>
 	  </collision>

File: bringup/urdf/tams_ur5_setup.urdf.xacro (robot description, xacro)
@@ -7,5 +7,5 @@
   <!-- arm -->
   <xacro:include filename="$(find tams_ur5_description)/urdf/arm.urdf.xacro" />
-  <xacro:include filename="$(find ur5_push_setup)/urdf/pusher.urdf.xacro" />
+  <xacro:include filename="$(find tams_ur5_push_bringup)/urdf/pusher.urdf.xacro" />
   <link name="world" />
   <joint name="world_floor_joint" type="fixed">
